File: Hardware/ESP32Shield.sch (EAGLE design)
At the start: 44 parts, among them J2 RJ45, J3 XLR-3-FEMALE, J4 XLR-3-MALE, U1 MAX3485CSA, U2 TXB0104

Commit message: post review changes
Parts:
- added FD1, FD2, FD3, FD4: FIDUCIALUFIDUCIAL, SparkFun-Aesthetics:FIDUCIALUFIDUCIAL
- added R10: 0, SparkFun-Resistors:0OHM-0603-1/10W-5%
- added TP1, TP2, TP3, TP4: TEST-POINT3, SparkFun-Connectors:TEST-POINT3
- R1: value 100 -> DNP
- renumbered U$1 to U3, U$2 to U4, U$3 to U5, U$4 to U6
Connections:
- net GND: now also R10.2
- net GND-ISO: now also R10.1
- net HV-DATA1: now also TP1.1
- net HV-DATA2: now also TP2.1
- net HV-DATA3: now also TP3.1
- net HV-LED-CLOCK: now also TP4.1
Other:
- note added: "Populate with a 120 Ohm resistor if this device is at the end of a DMX chain"
- note added: "Switch jumpers JP1 and JP2 to the other side of the jumper to enable RS-485 input"
- note added: "Vin: 5V"
- moved on the sheet: U2

Commit message: updating for reds
Parts:
- removed D1, D2, D3, D4: 3A/10V/280mV, SparkFun-DiscreteSemi:DIODE-SCHOTTKY-BAT60A
- removed J2: RJ45, SparkFun-Connectors:RJ45-8
- removed JP1, JP2: JUMPER-SMT_3_1-NC_PASTE_SILK, SparkFun-Jumpers:JUMPER-SMT_3_1-NC_PASTE_SILK
- removed R10: 0, SparkFun-Resistors:0OHM-0603-1/10W-5%
- LOGO1, LOGO2: value SFE_LOGO_NAME_FLAME.1_INCH -> SFE_LOGO_NAME_FLAME.2_INCH; device SparkFun-Aesthetics:SFE_LOGO_NAME_FLAME.1_INCH -> SparkFun-Aesthetics:SFE_LOGO_NAME_FLAME.2_INCH
Connections:
- removed net A-XLR: D1.C, J4.D-, JP1.3
- removed net B-XLR: D2.C, J4.D+, JP2.3
- removed net N$10: D2.A, J3.D+
- removed net N$11: D4.C, JP1.1
- removed net N$12: D3.C, JP2.1
- removed net N$7: D3.A, J2.1
- removed net N$8: D4.A, J2.2
- removed net N$9: D1.A, J3.D-
- net A: now also J3.D+, J4.D+; no longer JP2.2
- net B: now also J3.D-, J4.D-; no longer JP1.2
- net GND: no longer R10.2
- net GND-ISO: no longer R10.1
Other:
- note removed: "Switch jumpers JP1 and JP2 to the other side of the jumper to enable RS-485 input"
- moved on the sheet: J4
