File: Hardware/ESP32Shield.sch (EAGLE design)
At the start: 45 parts, among them J3 XLR-3-FEMALE, J4 XLR-3-MALE, U1 MAX3485CSA, U2 TXB0104, U3 6N137S, U4 6N137S, U5 6N137S, U6 RFB-0505S

Commit message: a few unsaved changes
Other:
- moved on the sheet: TP1, TP2, TP3, TP4
Changed lines of the file:
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@@
 <setting verticaltext="up"/>
 </settings>
-<grid distance="0.1" unitdist="inch" unit="inch" style="lines" multiple="1" display="no" altdistance="0.01" altunitdist="inch" altunit="inch"/>
+<grid distance="0.1" unitdist="inch" unit="inch" style="lines" multiple="1" display="no" altdistance="0.05" altunitdist="inch" altunit="inch"/>
 <layers>
 <layer number="1" name="Top" color="4" fill="1" visible="no" active="no"/>
@@
 <instance part="J1" gate="G$1" x="26.67" y="152.4"/>
 <instance part="J7" gate="G$1" x="26.67" y="157.48" rot="MR0"/>
-<instance part="SUPPLY7" gate="G$1" x="13.97" y="172.72"/>
+<instance part="SUPPLY7" gate="G$1" x="13.97" y="177.8"/>
 <instance part="SUPPLY8" gate="G$1" x="49.53" y="137.16"/>
 <instance part="U3" gate="G$1" x="154.94" y="124.46" rot="MR0"/>
@@
 <instance part="U6" gate="G$1" x="180.34" y="160.02"/>
 <instance part="SUPPLY1" gate="G$1" x="165.1" y="172.72"/>
-<instance part="GND1" gate="1" x="165.1" y="142.24"/>
-<instance part="GND-ISO1" gate="G$1" x="195.58" y="142.24"/>
+<instance part="GND1" gate="1" x="165.1" y="147.32"/>
+<instance part="GND-ISO1" gate="G$1" x="195.58" y="147.32"/>
 <instance part="U$5" gate="G$1" x="195.58" y="172.72"/>
 <instance part="C1" gate="G$1" x="154.94" y="162.56"/>
@@
 <instance part="FD3" gate="G$1" x="241.3" y="17.78"/>
 <instance part="FD4" gate="G$1" x="243.84" y="17.78"/>
-<instance part="TP1" gate="G$1" x="71.12" y="99.06" smashed="yes" rot="R90">
-<attribute name="NAME" x="71.12" y="96.52" size="1.778" layer="95" font="vector" rot="R90"/>
+<instance part="TP1" gate="G$1" x="71.12" y="101.6" smashed="yes" rot="R90">
+<attribute name="NAME" x="71.12" y="99.06" size="1.778" layer="95" font="vector" rot="R90"/>
 </instance>
-<instance part="TP2" gate="G$1" x="73.66" y="99.06" smashed="yes" rot="R90">
-<attribute name="NAME" x="73.66" y="96.52" size="1.778" layer="95" font="vector" rot="R90"/>
+<instance part="TP2" gate="G$1" x="73.66" y="101.6" smashed="yes" rot="R90">
+<attribute name="NAME" x="73.66" y="99.06" size="1.778" layer="95" font="vector" rot="R90"/>
 </instance>
-<instance part="TP3" gate="G$1" x="76.2" y="99.06" smashed="yes" rot="R90">
-<attribute name="NAME" x="76.2" y="96.52" size="1.778" layer="95" font="vector" rot="R90"/>
+<instance part="TP3" gate="G$1" x="76.2" y="101.6" smashed="yes" rot="R90">
+<attribute name="NAME" x="76.2" y="99.06" size="1.778" layer="95" font="vector" rot="R90"/>
 </instance>
-<instance part="TP4" gate="G$1" x="78.74" y="99.06" smashed="yes" rot="R90">
-<attribute name="NAME" x="78.74" y="96.52" size="1.778" layer="95" font="vector" rot="R90"/>
+<instance part="TP4" gate="G$1" x="78.74" y="101.6" smashed="yes" rot="R90">
+<attribute name="NAME" x="78.74" y="99.06" size="1.778" layer="95" font="vector" rot="R90"/>
 </instance>
 <instance part="SUPPLY12" gate="G$1" x="142.24" y="132.08"/>
@@
 <junction x="165.1" y="157.48"/>
 <pinref part="J12" gate="G$1" pin="1"/>
-<wire x1="165.1" y1="144.78" x2="165.1" y2="157.48" width="0.1524" layer="91"/>
+<wire x1="165.1" y1="149.86" x2="165.1" y2="157.48" width="0.1524" layer="91"/>
 <wire x1="147.32" y1="162.56" x2="149.86" y2="162.56" width="0.1524" layer="91"/>
 <wire x1="149.86" y1="162.56" x2="149.86" y2="157.48" width="0.1524" layer="91"/>
@@
 <pinref part="J7" gate="G$1" pin="3"/>
 <wire x1="16.51" y1="147.32" x2="13.97" y2="147.32" width="0.1524" layer="91"/>
-<wire x1="13.97" y1="147.32" x2="13.97" y2="172.72" width="0.1524" layer="91"/>
+<wire x1="13.97" y1="147.32" x2="13.97" y2="177.8" width="0.1524" layer="91"/>
 <pinref part="SUPPLY7" gate="G$1" pin="5V"/>
 </segment>
@@
 <junction x="195.58" y="157.48"/>
 <pinref part="C2" gate="G$1" pin="2"/>
-<wire x1="195.58" y1="144.78" x2="195.58" y2="157.48" width="0.1524" layer="91"/>
+<wire x1="195.58" y1="149.86" x2="195.58" y2="157.48" width="0.1524" layer="91"/>
 <wire x1="195.58" y1="157.48" x2="200.66" y2="157.48" width="0.1524" layer="91"/>
 <wire x1="200.66" y1="157.48" x2="200.66" y2="160.02" width="0.1524" layer="91"/>
@@
 <label x="81.28" y="93.98" size="1.27" layer="95" font="vector" xref="yes"/>
 <wire x1="73.66" y1="93.98" x2="81.28" y2="93.98" width="0.1524" layer="91"/>
-<wire x1="73.66" y1="93.98" x2="73.66" y2="99.06" width="0.1524" layer="91"/>
+<wire x1="73.66" y1="93.98" x2="73.66" y2="101.6" width="0.1524" layer="91"/>
 <junction x="73.66" y="93.98"/>
 <pinref part="TP2" gate="G$1" pin="1"/>
@@
 <label x="81.28" y="91.44" size="1.27" layer="95" font="vector" xref="yes"/>
 <wire x1="76.2" y1="91.44" x2="81.28" y2="91.44" width="0.1524" layer="91"/>
-<wire x1="76.2" y1="91.44" x2="76.2" y2="99.06" width="0.1524" layer="91"/>
+<wire x1="76.2" y1="91.44" x2="76.2" y2="101.6" width="0.1524" layer="91"/>
 <junction x="76.2" y="91.44"/>
 <pinref part="TP3" gate="G$1" pin="1"/>
@@
 <label x="81.28" y="96.52" size="1.27" layer="95" font="vector" xref="yes"/>
 <wire x1="71.12" y1="96.52" x2="81.28" y2="96.52" width="0.1524" layer="91"/>
-<wire x1="71.12" y1="96.52" x2="71.12" y2="99.06" width="0.1524" layer="91"/>
+<wire x1="71.12" y1="96.52" x2="71.12" y2="101.6" width="0.1524" layer="91"/>
 <junction x="71.12" y="96.52"/>
 <pinref part="TP1" gate="G$1" pin="1"/>
@@
 <label x="81.28" y="88.9" size="1.27" layer="95" font="vector" xref="yes"/>
 <wire x1="78.74" y1="88.9" x2="81.28" y2="88.9" width="0.1524" layer="91"/>
-<wire x1="78.74" y1="88.9" x2="78.74" y2="99.06" width="0.1524" layer="91"/>
+<wire x1="78.74" y1="88.9" x2="78.74" y2="101.6" width="0.1524" layer="91"/>
 <junction x="78.74" y="88.9"/>
 <pinref part="TP4" gate="G$1" pin="1"/>
